File: pcb/kitchen-timer.sch (KiCad schematic (older format))
At the start: 17 parts, among them J1 RT, J2 LCD, Q1 BC337, Q2 BC327, Q3 BC337, Q4 BC327, Q5 BC337

Commit message: add pcb
Parts:
- added D1: D, Diode_THT:D_A-405_P7.62mm_Horizontal, symbol Device:D_Small
- added IC1: ArduinoProMini, arduino:pro_mini, symbol mysensors_arduino:ArduinoProMini
- added J1: EX, Connector_PinHeader_1.27mm:PinHeader_1x02_P1.27mm_Vertical, symbol Connector:Conn_01x02_Male
- added J2: 3.3V, Connector_PinHeader_1.27mm:PinHeader_1x02_P1.27mm_Vertical, symbol Connector:Conn_01x02_Male
- added J4, J5: Conn_01x03, Connector_PinHeader_2.54mm:PinHeader_1x03_P2.54mm_Vertical, symbol Connector_Generic:Conn_01x03
- BT1: footprint (none) -> Connector_PinHeader_1.27mm:PinHeader_1x02_P1.27mm_Vertical
- BZ1: footprint (none) -> Buzzer_Beeper:Buzzer_12x9.5RM7.6
- C1, C2: footprint (none) -> Capacitor_THT:CP_Radial_D4.0mm_P2.00mm
- J3: renamed from J1; footprint (none) -> Connector_PinHeader_2.54mm:PinHeader_1x05_P2.54mm_Vertical
- J6: renamed from J2; footprint (none) -> Connector_PinHeader_2.54mm:PinHeader_1x04_P2.54mm_Vertical
- L1: footprint (none) -> Package_TO_SOT_THT:TO-92_Inline
- R1, R2, R3, R4: footprint (none) -> Resistor_THT:R_Axial_DIN0207_L6.3mm_D2.5mm_P10.16mm_Horizontal
- R5: footprint (none) -> Resistor_THT:R_Axial_DIN0204_L3.6mm_D1.6mm_P5.08mm_Horizontal
Connections:
- net +3V3: now also IC1.21 (VCC), J2.2 (Pin_2)
- net +9V: now also D1.2 (A); no longer BZ1.1 (-), C1.1, L1.2 (VIN)
- net -BATT: now also IC1.23 (GND), IC1.29 (GND), IC1.4 (GND), J1.2 (Pin_2), J2.1 (Pin_1)
- net BUZZER: now also IC1.13 ((PCINT2/OC1B/~SS~/PWM)PB2/10)
- net ENABLE_LCD: now also IC1.17 ((PCINT8/ADC0)PC0/14/A0)
- net ENABLE_RT: now also IC1.18 ((PCINT9/ADC1)PC1/15/A1)
- net LCD_CLK: now also IC1.11 ((PCINT0/CLKO/ICP1)PB0/8)
- net LCD_DIO: now also IC1.12 ((PCINT1/OC1A/PWM)PB1/9)
- net RT_CLK: now also IC1.6 ((PCINT19/OC2B/INT1/PWM)PD3/3)
- net RT_DT: now also IC1.10 ((PCINT23/AIN1)PD7/7)
- net RT_SW: now also IC1.5 ((PCINT18/INT0)PD2/2)
- new net: BZ1.1 (-), C1.1, D1.1 (K), J1.1 (Pin_1), L1.2 (VIN)
- new net: IC1.14 ((PCINT3/OC2A/MOSI/PWM)PB3/11), J4.1 (Pin_1)
- new net: IC1.15 ((PCINT4/MISO)PB4/12), J4.2 (Pin_2)
- new net: IC1.16 ((PCINT5/SCK)PB5/13), J4.3 (Pin_3)
- new net: IC1.7 ((PCINT20/XCK/T0)PD4/4), J5.1 (Pin_1)
- new net: IC1.8 ((PCINT21/OC0B/T1/PWM)PD5/5), J5.2 (Pin_2)
- new net: IC1.9 ((PCINT22/OC0A/AIN0/PWM)PD6/6), J5.3 (Pin_3)
- no-connect marks 0 -> 11

Commit message: add pcb
Parts:
- removed BT1: 9V, Connector_PinHeader_1.27mm:PinHeader_1x02_P1.27mm_Vertical, symbol Device:Battery_Cell
- removed C2: 10uF, Capacitor_THT:CP_Radial_D4.0mm_P2.00mm, symbol Device:CP1_Small
- removed D1: D, Diode_THT:D_A-405_P7.62mm_Horizontal, symbol Device:D_Small
- removed IC1: ArduinoProMini, arduino:pro_mini, symbol mysensors_arduino:ArduinoProMini
- removed J2: 3.3V, Connector_PinHeader_1.27mm:PinHeader_1x02_P1.27mm_Vertical, symbol Connector:Conn_01x02_Male
- removed J4, J5: Conn_01x03, Connector_PinHeader_2.54mm:PinHeader_1x03_P2.54mm_Vertical, symbol Connector_Generic:Conn_01x03
- removed L1: HT7333-A, Package_TO_SOT_THT:TO-92_Inline, symbol ht7333-a:HT7333-A
- removed Q2: BC327, Package_TO_SOT_THT:TO-92_Inline, symbol Transistor_BJT:BC327
- removed Q5: BC337, Package_TO_SOT_THT:TO-92_Inline, symbol Transistor_BJT:BC337
- added C2, C3: 100nf, Capacitor_SMD:C_0805_2012Metric_Pad1.15x1.40mm_HandSolder, symbol Device:C
- added J2: SW2, Connector_PinHeader_2.00mm:PinHeader_1x02_P2.00mm_Vertical, symbol Connector:Conn_01x02_Female
- added J5: LED1, Connector_PinHeader_2.00mm:PinHeader_1x02_P2.00mm_Vertical, symbol Connector:Conn_01x02_Female
- added U1: ATmega328-PU, Package_DIP:DIP-28_W7.62mm, symbol MCU_Microchip_ATmega:ATmega328-PU
- added Y1: 32khz, Crystal:Crystal_DS15_D1.5mm_L5.0mm_Vertical, symbol Device:Crystal_Small
- BZ1: footprint Buzzer_Beeper:Buzzer_12x9.5RM7.6 -> Connector_PinHeader_2.00mm:PinHeader_1x02_P2.00mm_Vertical
- J1: value EX -> USB_Breakout IN; footprint Connector_PinHeader_1.27mm:PinHeader_1x02_P1.27mm_Vertical -> Connector_PinHeader_2.00mm:PinHeader_1x02_P2.00mm_Vertical
- R1: value 2.6k -> 10k; footprint Resistor_THT:R_Axial_DIN0207_L6.3mm_D2.5mm_P10.16mm_Horizontal -> Resistor_SMD:R_0805_2012Metric_Pad1.15x1.40mm_HandSolder
- R2, R3, R4: footprint Resistor_THT:R_Axial_DIN0207_L6.3mm_D2.5mm_P10.16mm_Horizontal -> Resistor_SMD:R_0805_2012Metric_Pad1.15x1.40mm_HandSolder
- R5: value 2.6k -> 220; footprint Resistor_THT:R_Axial_DIN0204_L3.6mm_D1.6mm_P5.08mm_Horizontal -> Resistor_THT:R_Axial_DIN0207_L6.3mm_D2.5mm_P10.16mm_Horizontal
- renumbered J6 to J4, Q3 to Q2, Q4 to Q3
Connections:
- net +3V3: now also BZ1.1 (-), C1.1, J1.1 (Pin_1), J3.2 (Pin_2), R1.1, C2.1, C3.1, U1.20 (AVCC), U1.21 (AREF), U1.7 (VCC)
- net ENABLE_LCD: now also U1.23 (PC0)
- net LCD_CLK: now also U1.14 (PB0)
- net LCD_DIO: now also U1.15 (PB1)
- net RT_CLK: now also U1.5 (PD3)
- net RT_DT: now also U1.13 (PD7)
- net RT_SW: now also U1.4 (PD2)
- net at BZ1.2 (+): now also Q1.1 (C)
- net at R5.1: now also U1.25 (PC2)
- net at R2.2: now also U1.12 (PD6); no longer Q1.1 (C)
- net at Q1.2 (B): now also R2.1; no longer R1.1
- net -BATT renamed GND
- net GND: now also C2.2, C3.2, J2.2 (Pin_2), J5.1 (Pin_1), U1.22 (GND), U1.8 (GND)
- net BUZZER: no longer names the net of R5.2
- net BUZZER: now also J5.2 (Pin_2)
- net ENABLE_RT: no longer names the net of R1.2
- net ENABLE_RT: now also U1.1 (~RESET~/PC6)
- new net: U1.10 (XTAL2/PB7), Y1.2
- new net: J2.1 (Pin_1), U1.24 (PC1)
- new net: U1.9 (XTAL1/PB6), Y1.1
- no-connect marks 11 -> 0
Other:
- moved on the sheet: BZ1
